Commit message: add vaccum gripper

File: drone_description/urdf/vaccum_gripper.xacro (robot description, xacro)
@@ -12,7 +12,7 @@
       </xacro:cylinder_inertial_with_origin>
       <collision>
-        <origin xyz="0 0 0.015" rpy="0 0 0" />
+        <origin xyz="0 0 0" rpy="0 0 0" />
         <geometry>
-          <cylinder radius="0.02" length="0.03"/>
+          <cylinder radius="0.2" length="0.07"/>
         </geometry>
         <surface>
@@ -26,7 +26,7 @@
       </collision>
       <visual>
-        <origin xyz="0 0 0" rpy="0 0 0" />
+        <origin xyz="0 0 -0.025" rpy="0 0 0" />
         <geometry>
-          <cylinder radius="0.02" length="0.06"/>
+          <cylinder radius="0.02" length="0.05"/>
         </geometry>
         <material name="red"/>
