Commit message: add tilt_camera

File: drone_description/urdf/gimbal_camera.xacro (robot description, xacro)
@@ -130,4 +130,98 @@
       </xacro:cylinder_inertial_with_origin>
       <origin xyz="0 0 0" rpy="${pi/2} ${-pi/2} 0" />
+    </xacro:camera_with_inertial_macro>
+  </xacro:macro>
+  <xacro:macro name="tilt_camera_macro" params="namespace parent_link frame_rate
+      horizontal_fov image_width image_height image_format min_distance
+      max_distance noise_mean noise_stddev offset *origin">
+    <gazebo>
+      <plugin name="gazebo_ros_control" filename="libgazebo_ros_control.so">
+        <robotNamespace>${namespace}</robotNamespace>
+        <robotSimType>gazebo_ros_control/DefaultRobotHWSim</robotSimType>
+        <legacyModeNS>true</legacyModeNS>
+      </plugin>
+    </gazebo>
+    <joint name="${namespace}/gimbal_base_joint" type="fixed">
+      <xacro:insert_block name="origin" />
+      <parent link="${parent_link}"/>
+      <child link="${namespace}/gimbal_base_link"/>
+    </joint>
+    <link name="${namespace}/gimbal_base_link">
+      <xacro:box_inertial_with_origin
+        x="0.005"
+        y="0.02"
+        z="${offset + 0.01}"
+        mass="0.06">
+        <origin xyz="0.0 0.02 ${(offset + 0.01) / 2.0}" rpy="0 0 0"/>
+      </xacro:box_inertial_with_origin>
+      <visual>
+        <origin xyz="0.0 0.02 ${(offset + 0.01) / 2.0}" rpy="0 0 0" />
+        <geometry>
+          <box size="0.005 0.02 ${offset + 0.01}"/>
+        </geometry>
+        <material name="blue"/>
+      </visual>
+    </link>
+    <joint name="${namespace}/gimbal_pitch_joint" type="revolute">
+      <origin xyz="0.0 0.0 ${offset}" rpy="${pi} 0.0 0.0"/>
+      <parent link="${namespace}/gimbal_base_link"/>
+      <child link="${namespace}/gimbal_pitch_link"/>
+      <axis xyz="0.0 1.0 0.0"/>
+      <limit lower="${-pi/4}" upper="${pi/4}" effort="0.2" velocity="6.0"/>
+    </joint>
+    <link name="${namespace}/gimbal_pitch_link">
+      <xacro:box_inertial_with_origin
+        x="0.005"
+        y="0.03"
+        z="0.02"
+        mass="0.01">
+        <origin xyz="0.0 0.025 0.0" rpy="0 0 0" />
+      </xacro:box_inertial_with_origin>
+      <visual>
+        <origin xyz="0.0 0.025 0.0" rpy="0 0 0" />
+        <geometry>
+          <box size="0.005 0.03 0.02"/>
+        </geometry>
+        <material name="green"/>
+      </visual>
+    </link>
+    <transmission name="${namespace}/pitch_tran">
+      <type>transmission_interface/SimpleTransmission</type>
+      <joint name="${namespace}/gimbal_pitch_joint">
+        <hardwareInterface>hardware_interface/EffortJointInterface</hardwareInterface>
+      </joint>
+      <actuator name="${namespace}/gimbal_pitch_motor">
+        <hardwareInterface>hardware_interface/EffortJointInterface</hardwareInterface>
+        <mechanicalReduction>1</mechanicalReduction>
+      </actuator>
+    </transmission>
+    <gazebo reference="${namespace}/gimbal_base_link">
+      <material>Gazebo/Blue</material>
+    </gazebo>
+    <gazebo reference="${namespace}/gimbal_pitch_link">
+      <material>Gazebo/Green</material>
+    </gazebo>
+    <xacro:camera_with_inertial_macro
+      namespace="${namespace}"
+      parent_link="${namespace}/gimbal_pitch_link"
+      camera_suffix="0"
+      frame_rate="${frame_rate}"
+      horizontal_fov="${horizontal_fov}"
+      image_width="${image_width}"
+      image_height="${image_height}"
+      image_format="${image_format}"
+      min_distance="${min_distance}"
+      max_distance="${max_distance}"
+      noise_mean="${noise_mean}"
+      noise_stddev="${noise_stddev}"
+      enable_visual="true">
+      <cylinder radius="0.01" length="0.005"/>
+      <xacro:cylinder_inertial_with_origin
+        radius="0.01"
+        length="0.005"
+        mass="0.12">
+        <origin xyz="0 0 0" rpy="${-pi} 0 0" />
+      </xacro:cylinder_inertial_with_origin>
+      <origin xyz="0 0 0" rpy="${-pi} 0 0" />
     </xacro:camera_with_inertial_macro>
   </xacro:macro>

Commit message: update

File: drone_description/urdf/gimbal_camera.xacro (robot description, xacro)
@@ -152,5 +152,5 @@
         y="0.02"
         z="${offset + 0.01}"
-        mass="0.06">
+        mass="0.0001">
         <origin xyz="0.0 0.02 ${(offset + 0.01) / 2.0}" rpy="0 0 0"/>
       </xacro:box_inertial_with_origin>
@@ -168,5 +168,5 @@
       <child link="${namespace}/gimbal_pitch_link"/>
       <axis xyz="0.0 1.0 0.0"/>
-      <limit lower="${-pi/4}" upper="${pi/4}" effort="0.2" velocity="6.0"/>
+      <limit lower="${-pi/3}" upper="${pi/3}" effort="0.2" velocity="6"/>
     </joint>
     <link name="${namespace}/gimbal_pitch_link">
@@ -175,5 +175,5 @@
         y="0.03"
         z="0.02"
-        mass="0.01">
+        mass="0.0001">
         <origin xyz="0.0 0.025 0.0" rpy="0 0 0" />
       </xacro:box_inertial_with_origin>
@@ -186,14 +186,4 @@
       </visual>
     </link>
-    <transmission name="${namespace}/pitch_tran">
-      <type>transmission_interface/SimpleTransmission</type>
-      <joint name="${namespace}/gimbal_pitch_joint">
-        <hardwareInterface>hardware_interface/EffortJointInterface</hardwareInterface>
-      </joint>
-      <actuator name="${namespace}/gimbal_pitch_motor">
-        <hardwareInterface>hardware_interface/EffortJointInterface</hardwareInterface>
-        <mechanicalReduction>1</mechanicalReduction>
-      </actuator>
-    </transmission>
     <gazebo reference="${namespace}/gimbal_base_link">
       <material>Gazebo/Blue</material>
@@ -220,5 +210,5 @@
         radius="0.01"
         length="0.005"
-        mass="0.12">
+        mass="0.0001">
         <origin xyz="0 0 0" rpy="${-pi} 0 0" />
       </xacro:cylinder_inertial_with_origin>

Commit message: latest stable

File: drone_description/urdf/gimbal_camera.xacro (robot description, xacro)
@@ -26,7 +26,21 @@
       </xacro:box_inertial_with_origin>
       <visual>
+        <origin xyz="0.0 -0.02625 0" rpy="0 0 0" />
+        <geometry>
+          <box size="0.015 0.0525 0.005"/>
+        </geometry>
+        <material name="blue"/>
+      </visual>
+      <visual>
         <origin xyz="0.0 -0.05 -${offset / 2.0}" rpy="0 0 0" />
         <geometry>
-          <box size="0.02 0.005 ${offset}"/>
+          <box size="0.015 0.005 ${offset}"/>
+        </geometry>
+        <material name="blue"/>
+      </visual>
+      <visual>
+        <origin xyz="0.0 -0.05 -${offset}" rpy="${pi / 2.0} 0 0" />
+        <geometry>
+          <cylinder radius="0.01" length="0.01"/>
         </geometry>
         <material name="blue"/>
@@ -49,17 +63,31 @@
       </xacro:box_inertial_with_origin>
       <visual>
-        <origin xyz="0 -0.02 0.0" rpy="0 0 0" />
-        <geometry>
-          <box size="0.02 0.04 0.005"/>
+        <origin xyz="-0.02 -0.0075 0.0" rpy="0 0 0" />
+        <geometry>
+          <box size="0.06 0.005 0.015"/>
         </geometry>
         <material name="green"/>
       </visual>
+      <visual>
+        <origin xyz="-0.05 -0.0275 0.0" rpy="0 0 0" />
+        <geometry>
+          <box size="0.005 0.045 0.015"/>
+        </geometry>
+        <material name="green"/>
+      </visual>
+      <visual>
+        <origin xyz="-0.05 -0.05 0" rpy="0 ${pi / 2.0} 0" />
+        <geometry>
+          <cylinder radius="0.01" length="0.01"/>
+        </geometry>
+        <material name="green"/>
+      </visual>
     </link>
     <joint name="${namespace}/gimbal_roll_joint" type="revolute">
-      <origin xyz="0 -0.05 0.0" rpy="0.0 0.0 0.0"/>
+      <origin xyz="-0.05 -0.05 0.0" rpy="0.0 0.0 0.0"/>
       <parent link="${namespace}/gimbal_pitch_link"/>
       <child link="${namespace}/gimbal_roll_link"/>
       <axis xyz="1.0 0.0 0.0"/>
-      <limit lower="${-pi/4}" upper="${pi/4}" effort="0.2" velocity="6.0"/>
+      <limit lower="${-pi/4}" upper="${pi/4}" effort="1.2" velocity="6.0"/>
     </joint>
     <link name="${namespace}/gimbal_roll_link">
@@ -69,10 +97,10 @@
         z="0.005"
         mass="0.06">
-        <origin xyz="-0.025 0 0" rpy="0 0 0" />
+        <origin xyz="0.025 0 0" rpy="0 0 0" />
       </xacro:box_inertial_with_origin>
       <visual>
-        <origin xyz="-0.025 0 0" rpy="0 0 0" />
-        <geometry>
-          <box size="0.03 0.02 0.005"/>
+        <origin xyz="0.0275 0 0" rpy="0 0 0" />
+        <geometry>
+          <box size="0.045 0.015 0.005"/>
         </geometry>
         <material name="red"/>
@@ -122,5 +150,5 @@
       noise_stddev="${noise_stddev}"
       enable_visual="true">
-      <cylinder radius="0.01" length="0.005"/>
+      <cylinder radius="0.01" length="0.006"/>
       <xacro:cylinder_inertial_with_origin
         radius="0.01"
@@ -129,89 +157,5 @@
         <origin xyz="0 0 0" rpy="0 0 0" />
       </xacro:cylinder_inertial_with_origin>
-      <origin xyz="0 0 0" rpy="${pi/2} ${-pi/2} 0" />
-    </xacro:camera_with_inertial_macro>
-  </xacro:macro>
-  <xacro:macro name="tilt_camera_macro" params="namespace parent_link frame_rate
-      horizontal_fov image_width image_height image_format min_distance
-      max_distance noise_mean noise_stddev offset *origin">
-    <gazebo>
-      <plugin name="gazebo_ros_control" filename="libgazebo_ros_control.so">
-        <robotNamespace>${namespace}</robotNamespace>
-        <robotSimType>gazebo_ros_control/DefaultRobotHWSim</robotSimType>
-        <legacyModeNS>true</legacyModeNS>
-      </plugin>
-    </gazebo>
-    <joint name="${namespace}/gimbal_base_joint" type="fixed">
-      <xacro:insert_block name="origin" />
-      <parent link="${parent_link}"/>
-      <child link="${namespace}/gimbal_base_link"/>
-    </joint>
-    <link name="${namespace}/gimbal_base_link">
-      <xacro:box_inertial_with_origin
-        x="0.005"
-        y="0.02"
-        z="${offset + 0.01}"
-        mass="0.0001">
-        <origin xyz="0.0 0.02 ${(offset + 0.01) / 2.0}" rpy="0 0 0"/>
-      </xacro:box_inertial_with_origin>
-      <visual>
-        <origin xyz="0.0 0.02 ${(offset + 0.01) / 2.0}" rpy="0 0 0" />
-        <geometry>
-          <box size="0.005 0.02 ${offset + 0.01}"/>
-        </geometry>
-        <material name="blue"/>
-      </visual>
-    </link>
-    <joint name="${namespace}/gimbal_pitch_joint" type="revolute">
-      <origin xyz="0.0 0.0 ${offset}" rpy="${pi} 0.0 0.0"/>
-      <parent link="${namespace}/gimbal_base_link"/>
-      <child link="${namespace}/gimbal_pitch_link"/>
-      <axis xyz="0.0 1.0 0.0"/>
-      <limit lower="${-pi/3}" upper="${pi/3}" effort="0.2" velocity="6"/>
-    </joint>
-    <link name="${namespace}/gimbal_pitch_link">
-      <xacro:box_inertial_with_origin
-        x="0.005"
-        y="0.03"
-        z="0.02"
-        mass="0.0001">
-        <origin xyz="0.0 0.025 0.0" rpy="0 0 0" />
-      </xacro:box_inertial_with_origin>
-      <visual>
-        <origin xyz="0.0 0.025 0.0" rpy="0 0 0" />
-        <geometry>
-          <box size="0.005 0.03 0.02"/>
-        </geometry>
-        <material name="green"/>
-      </visual>
-    </link>
-    <gazebo reference="${namespace}/gimbal_base_link">
-      <material>Gazebo/Blue</material>
-    </gazebo>
-    <gazebo reference="${namespace}/gimbal_pitch_link">
-      <material>Gazebo/Green</material>
-    </gazebo>
-    <xacro:camera_with_inertial_macro
-      namespace="${namespace}"
-      parent_link="${namespace}/gimbal_pitch_link"
-      camera_suffix="0"
-      frame_rate="${frame_rate}"
-      horizontal_fov="${horizontal_fov}"
-      image_width="${image_width}"
-      image_height="${image_height}"
-      image_format="${image_format}"
-      min_distance="${min_distance}"
-      max_distance="${max_distance}"
-      noise_mean="${noise_mean}"
-      noise_stddev="${noise_stddev}"
-      enable_visual="true">
-      <cylinder radius="0.01" length="0.005"/>
-      <xacro:cylinder_inertial_with_origin
-        radius="0.01"
-        length="0.005"
-        mass="0.0001">
-        <origin xyz="0 0 0" rpy="${-pi} 0 0" />
-      </xacro:cylinder_inertial_with_origin>
-      <origin xyz="0 0 0" rpy="${-pi} 0 0" />
+      <origin xyz="0.05 0 0" rpy="${pi/2} ${-pi/2} 0" />
     </xacro:camera_with_inertial_macro>
   </xacro:macro>

Commit message: update

File: drone_description/urdf/gimbal_camera.xacro (robot description, xacro)
@@ -47,12 +47,14 @@
       </visual>
     </link>
-    <joint name="${namespace}/gimbal_pitch_joint" type="revolute">
-      <origin xyz="0.0 -0.05 -${offset}" rpy="${pi} 0.0 0.0"/>
-      <parent link="${namespace}/gimbal_base_link"/>
-      <child link="${namespace}/gimbal_pitch_link"/>
+    <xacro:revolute_gimbal_joint_macro
+      namespace="${namespace}"
+      joint_suffix="0"
+      parent_link="${namespace}/gimbal_base_link"
+      child_link="${namespace}/gimbal_tilt_link">
       <axis xyz="0.0 1.0 0.0"/>
       <limit lower="${-pi/4}" upper="${pi/4}" effort="0.2" velocity="6.0"/>
-    </joint>
-    <link name="${namespace}/gimbal_pitch_link">
+      <origin xyz="0.0 -0.05 -${offset}" rpy="${pi} 0.0 0.0"/>
+    </xacro:revolute_gimbal_joint_macro>
+    <link name="${namespace}/gimbal_tilt_link">
       <xacro:box_inertial_with_origin
         x="0.02"
@@ -84,12 +86,14 @@
       </visual>
     </link>
-    <joint name="${namespace}/gimbal_roll_joint" type="revolute">
-      <origin xyz="-0.05 -0.05 0.0" rpy="0.0 0.0 0.0"/>
-      <parent link="${namespace}/gimbal_pitch_link"/>
-      <child link="${namespace}/gimbal_roll_link"/>
+    <xacro:revolute_gimbal_joint_macro
+      namespace="${namespace}"
+      joint_suffix="1"
+      parent_link="${namespace}/gimbal_tilt_link"
+      child_link="${namespace}/gimbal_pan_link">
       <axis xyz="1.0 0.0 0.0"/>
       <limit lower="${-pi/4}" upper="${pi/4}" effort="1.2" velocity="6.0"/>
-    </joint>
-    <link name="${namespace}/gimbal_roll_link">
+      <origin xyz="-0.05 -0.05 0.0" rpy="0.0 0.0 0.0"/>
+    </xacro:revolute_gimbal_joint_macro>
+    <link name="${namespace}/gimbal_pan_link">
       <xacro:box_inertial_with_origin
         x="0.03"
@@ -107,36 +111,16 @@
       </visual>
     </link>
-    <transmission name="${namespace}/pitch_tran">
-      <type>transmission_interface/SimpleTransmission</type>
-      <joint name="${namespace}/gimbal_pitch_joint">
-        <hardwareInterface>hardware_interface/EffortJointInterface</hardwareInterface>
-      </joint>
-      <actuator name="${namespace}/gimbal_pitch_motor">
-        <hardwareInterface>hardware_interface/EffortJointInterface</hardwareInterface>
-        <mechanicalReduction>1</mechanicalReduction>
-      </actuator>
-    </transmission>
-    <transmission name="${namespace}/roll_tran">
-      <type>transmission_interface/SimpleTransmission</type>
-      <joint name="${namespace}/gimbal_roll_joint">
-        <hardwareInterface>hardware_interface/EffortJointInterface</hardwareInterface>
-      </joint>
-      <actuator name="${namespace}/gimbal_roll_motor">
-        <hardwareInterface>hardware_interface/EffortJointInterface</hardwareInterface>
-        <mechanicalReduction>1</mechanicalReduction>
-      </actuator>
-    </transmission>
     <gazebo reference="${namespace}/gimbal_base_link">
       <material>Gazebo/Blue</material>
     </gazebo>
-    <gazebo reference="${namespace}/gimbal_pitch_link">
+    <gazebo reference="${namespace}/gimbal_tilt_link">
       <material>Gazebo/Green</material>
     </gazebo>
-    <gazebo reference="${namespace}/gimbal_roll_link">
+    <gazebo reference="${namespace}/gimbal_pan_link">
       <material>Gazebo/Red</material>
     </gazebo>
     <xacro:camera_with_inertial_macro
       namespace="${namespace}"
-      parent_link="${namespace}/gimbal_roll_link"
+      parent_link="${namespace}/gimbal_pan_link"
       camera_suffix="0"
       frame_rate="${frame_rate}"
@@ -159,4 +143,24 @@
       <origin xyz="0.05 0 0" rpy="${pi/2} ${-pi/2} 0" />
     </xacro:camera_with_inertial_macro>
+  </xacro:macro>
+  <xacro:macro name="revolute_gimbal_joint_macro"
+    params="namespace joint_suffix parent_link child_link *axis *limit *origin">
+    <joint name="${namespace}/gimbal_joint_${joint_suffix}" type="revolute">
+      <parent link="${parent_link}"/>
+      <child link="${child_link}"/>
+      <xacro:insert_block name="axis" />
+      <xacro:insert_block name="limit" />
+      <xacro:insert_block name="origin" />
+    </joint>
+    <transmission name="${namespace}/gimbal_joint_trans_${joint_suffix}">
+      <type>transmission_interface/SimpleTransmission</type>
+      <joint name="${namespace}/gimbal_joint_${joint_suffix}">
+        <hardwareInterface>hardware_interface/EffortJointInterface</hardwareInterface>
+      </joint>
+      <actuator name="${namespace}/gimbal_joint_motor_${joint_suffix}">
+        <hardwareInterface>hardware_interface/EffortJointInterface</hardwareInterface>
+        <mechanicalReduction>1</mechanicalReduction>
+      </actuator>
+    </transmission>
   </xacro:macro>
   <xacro:macro name="camera_with_inertial_macro"

Commit message: add distort camera

File: drone_description/urdf/gimbal_camera.xacro (robot description, xacro)
@@ -4,5 +4,5 @@
   <xacro:macro name="pan_tilt_camera_macro" params="namespace parent_link frame_rate
       horizontal_fov image_width image_height image_format min_distance
-      max_distance noise_mean noise_stddev offset *origin">
+      max_distance noise_mean noise_stddev k1 k2 k3 p1 p2 cx cy offset enable_visual *origin">
     <gazebo>
       <plugin name="gazebo_ros_control" filename="libgazebo_ros_control.so">
@@ -120,5 +120,5 @@
       <material>Gazebo/Red</material>
     </gazebo>
-    <xacro:camera_with_inertial_macro
+    <xacro:camera_with_distortion_macro
       namespace="${namespace}"
       parent_link="${namespace}/gimbal_pan_link"
@@ -133,6 +133,12 @@
       noise_mean="${noise_mean}"
       noise_stddev="${noise_stddev}"
-      enable_visual="true">
-      <cylinder radius="0.01" length="0.006"/>
+      enable_visual="${enable_visual}"
+      k1="${k1}"
+      k2="${k2}"
+      k3="${k3}"
+      p1="${p1}"
+      p2="${p2}"
+      cx="${cx}"
+      cy="${cy}">
       <xacro:cylinder_inertial_with_origin
         radius="0.01"
@@ -142,5 +148,5 @@
       </xacro:cylinder_inertial_with_origin>
       <origin xyz="0.05 0 0" rpy="${pi/2} ${-pi/2} 0" />
-    </xacro:camera_with_inertial_macro>
+    </xacro:camera_with_distortion_macro>
   </xacro:macro>
   <xacro:macro name="revolute_gimbal_joint_macro"
@@ -164,24 +170,9 @@
     </transmission>
   </xacro:macro>
-  <xacro:macro name="camera_with_inertial_macro"
+  <xacro:macro name="camera_with_distortion_macro"
     params="namespace parent_link camera_suffix frame_rate
       horizontal_fov image_width image_height image_format min_distance
-      max_distance noise_mean noise_stddev enable_visual *geometry *inertial *origin">
+      max_distance noise_mean noise_stddev enable_visual k1 k2 k3 p1 p2 cx cy *inertial *origin">
     <link name="${namespace}/camera_${camera_suffix}_link">
-      <collision>
-        <origin xyz="0 0 0" rpy="0 0 0" />
-        <geometry>
-          <xacro:insert_block name="geometry" />
-        </geometry>
-      </collision>
-      <xacro:if value="${enable_visual}">
-        <visual>
-          <origin xyz="0 0 0" rpy="0 ${pi/2} 0" />
-          <geometry>
-            <xacro:insert_block name="geometry" />
-          </geometry>
-          <material name="orange" />
-        </visual>
-      </xacro:if>
       <xacro:insert_block name="inertial" />
     </link>
@@ -199,6 +190,5 @@
     <gazebo reference="${namespace}/camera_${camera_suffix}_link">
       <material>Gazebo/Orange</material>
-      <sensor type="camera" name="${namespace}_camera_${camera_suffix}">
-        <update_rate>${frame_rate}</update_rate>
+      <sensor type="camera" name="camera_${camera_suffix}">
         <camera name="head">
           <horizontal_fov>${horizontal_fov}</horizontal_fov>
@@ -212,4 +202,12 @@
             <far>${max_distance}</far>
           </clip>
+          <distortion>
+            <k1>${k1}</k1>
+            <k2>${k2}</k2>
+            <k3>${k3}</k3>
+            <p1>${p1}</p1>
+            <p2>${p2}</p2>
+            <center>${cx} ${cy}</center>
+          </distortion>
           <noise>
             <type>gaussian</type>
@@ -221,18 +219,15 @@
           </noise>
         </camera>
-        <plugin name="${namespace}_camera_${camera_suffix}_controller" filename="libgazebo_ros_camera.so">
+        <always_on>true</always_on>
+        <update_rate>${frame_rate}</update_rate>
+        <xacro:if value="${enable_visual}">
+          <visualize>true</visualize>
+        </xacro:if>
+        <plugin name="${namespace}_${camera_suffix}_controller" filename="libgazebo_ros_camera.so">
           <robotNamespace>${namespace}</robotNamespace>
-          <alwaysOn>true</alwaysOn>
-          <updateRate>${frame_rate}</updateRate>
           <cameraName>camera_${camera_suffix}</cameraName>
           <imageTopicName>image_raw</imageTopicName>
           <cameraInfoTopicName>camera_info</cameraInfoTopicName>
           <frameName>camera_${camera_suffix}_link</frameName>
-          <hackBaseline>0.0</hackBaseline>
-          <distortionK1>0.0</distortionK1>
-          <distortionK2>0.0</distortionK2>
-          <distortionK3>0.0</distortionK3>
-          <distortionT1>0.0</distortionT1>
-          <distortionT2>0.0</distortionT2>
         </plugin>
       </sensor>
