Commit message: add 3-axis gimbal camera

File: drone_description/urdf/gimbal_camera.xacro (robot description, xacro)
@@ -2,4 +2,169 @@
 <robot xmlns:xacro="http://ros.org/wiki/xacro">
   <xacro:include filename="$(find drone_description)/urdf/common.xacro" />
+  <xacro:macro name="gimbal_camera_macro" params="namespace parent_link frame_rate
+      horizontal_fov image_width image_height image_format min_distance
+      max_distance noise_mean noise_stddev k1 k2 k3 p1 p2 cx cy offset enable_visual *origin">
+    <gazebo>
+      <plugin name="gazebo_ros_control" filename="libgazebo_ros_control.so">
+        <robotNamespace>${namespace}</robotNamespace>
+        <robotSimType>gazebo_ros_control/DefaultRobotHWSim</robotSimType>
+        <legacyModeNS>true</legacyModeNS>
+      </plugin>
+    </gazebo>
+    <joint name="${namespace}/gimbal_base_joint" type="fixed">
+      <xacro:insert_block name="origin" />
+      <parent link="${parent_link}"/>
+      <child link="${namespace}/gimbal_base_link"/>
+    </joint>
+    <link name="${namespace}/gimbal_base_link">
+      <xacro:cylinder_inertial_with_origin
+        radius="0.01"
+        length="0.01"
+        mass="0.001">
+        <origin xyz="0 0 0" rpy="0 0 0" />
+      </xacro:cylinder_inertial_with_origin>
+    </link>
+    <xacro:revolute_gimbal_joint_macro
+      namespace="${namespace}"
+      joint_suffix="0"
+      parent_link="${namespace}/gimbal_base_link"
+      child_link="${namespace}/gimbal_link_0">
+      <axis xyz="0.0 0.0 1.0"/>
+      <limit lower="${-pi/2}" upper="${pi/2}" effort="1.2" velocity="6.0"/>
+      <origin xyz="0.0 0.0 0.0" rpy="0.0 0.0 -1.57"/>
+    </xacro:revolute_gimbal_joint_macro>
+    <link name="${namespace}/gimbal_link_0">
+      <xacro:box_inertial_with_origin
+        x="0.02"
+        y="0.005"
+        z="${offset}"
+        mass="0.06">
+        <origin xyz="0.0 -0.05 -${offset / 2.0}" rpy="0 0 0"/>
+      </xacro:box_inertial_with_origin>
+      <visual>
+        <origin xyz="0.0 -0.02625 0" rpy="0 0 0" />
+        <geometry>
+          <box size="0.015 0.0525 0.005"/>
+        </geometry>
+        <material name="blue"/>
+      </visual>
+      <visual>
+        <origin xyz="0.0 -0.05 -${offset / 2.0}" rpy="0 0 0" />
+        <geometry>
+          <box size="0.015 0.005 ${offset}"/>
+        </geometry>
+        <material name="blue"/>
+      </visual>
+      <visual>
+        <origin xyz="0.0 -0.05 -${offset}" rpy="${pi / 2.0} 0 0" />
+        <geometry>
+          <cylinder radius="0.01" length="0.01"/>
+        </geometry>
+        <material name="blue"/>
+      </visual>
+    </link>
+    <xacro:revolute_gimbal_joint_macro
+      namespace="${namespace}"
+      joint_suffix="1"
+      parent_link="${namespace}/gimbal_link_0"
+      child_link="${namespace}/gimbal_link_1">
+      <axis xyz="0.0 -1.0 0.0"/>
+      <limit lower="${-pi/4}" upper="${pi/4}" effort="0.2" velocity="6.0"/>
+      <origin xyz="0.0 -0.05 -${offset}" rpy="${pi} 0.0 0.0"/>
+    </xacro:revolute_gimbal_joint_macro>
+    <link name="${namespace}/gimbal_link_1">
+      <xacro:box_inertial_with_origin
+        x="0.02"
+        y="0.04"
+        z="0.005"
+        mass="0.06">
+        <origin xyz="0 -0.02 0.0" rpy="0 0 0" />
+      </xacro:box_inertial_with_origin>
+      <visual>
+        <origin xyz="-0.02 -0.0075 0.0" rpy="0 0 0" />
+        <geometry>
+          <box size="0.06 0.005 0.015"/>
+        </geometry>
+        <material name="green"/>
+      </visual>
+      <visual>
+        <origin xyz="-0.05 -0.0275 0.0" rpy="0 0 0" />
+        <geometry>
+          <box size="0.005 0.045 0.015"/>
+        </geometry>
+        <material name="green"/>
+      </visual>
+      <visual>
+        <origin xyz="-0.05 -0.05 0" rpy="0 ${pi / 2.0} 0" />
+        <geometry>
+          <cylinder radius="0.01" length="0.01"/>
+        </geometry>
+        <material name="green"/>
+      </visual>
+    </link>
+    <xacro:revolute_gimbal_joint_macro
+      namespace="${namespace}"
+      joint_suffix="2"
+      parent_link="${namespace}/gimbal_link_1"
+      child_link="${namespace}/gimbal_link_2">
+      <axis xyz="-1.0 0.0 0.0"/>
+      <limit lower="${-pi/4}" upper="${pi/4}" effort="1.2" velocity="6.0"/>
+      <origin xyz="-0.05 -0.05 0.0" rpy="0.0 0.0 0.0"/>
+    </xacro:revolute_gimbal_joint_macro>
+    <link name="${namespace}/gimbal_link_2">
+      <xacro:box_inertial_with_origin
+        x="0.03"
+        y="0.02"
+        z="0.005"
+        mass="0.06">
+        <origin xyz="0.025 0 0" rpy="0 0 0" />
+      </xacro:box_inertial_with_origin>
+      <visual>
+        <origin xyz="0.0275 0 0" rpy="0 0 0" />
+        <geometry>
+          <box size="0.045 0.015 0.005"/>
+        </geometry>
+        <material name="red"/>
+      </visual>
+    </link>
+    <gazebo reference="${namespace}/gimbal_link_0">
+      <material>Gazebo/Blue</material>
+    </gazebo>
+    <gazebo reference="${namespace}/gimbal_link_1">
+      <material>Gazebo/Green</material>
+    </gazebo>
+    <gazebo reference="${namespace}/gimbal_link_2">
+      <material>Gazebo/Red</material>
+    </gazebo>
+    <xacro:camera_with_distortion_macro
+      namespace="${namespace}"
+      parent_link="${namespace}/gimbal_link_2"
+      camera_suffix="0"
+      frame_rate="${frame_rate}"
+      horizontal_fov="${horizontal_fov}"
+      image_width="${image_width}"
+      image_height="${image_height}"
+      image_format="${image_format}"
+      min_distance="${min_distance}"
+      max_distance="${max_distance}"
+      noise_mean="${noise_mean}"
+      noise_stddev="${noise_stddev}"
+      enable_visual="${enable_visual}"
+      k1="${k1}"
+      k2="${k2}"
+      k3="${k3}"
+      p1="${p1}"
+      p2="${p2}"
+      cx="${cx}"
+      cy="${cy}">
+      <xacro:cylinder_inertial_with_origin
+        radius="0.01"
+        length="0.005"
+        mass="0.12">
+        <origin xyz="0 0 0" rpy="0 0 0" />
+      </xacro:cylinder_inertial_with_origin>
+      <origin xyz="0.05 0 0" rpy="${pi/2} ${-pi/2} 0" />
+    </xacro:camera_with_distortion_macro>
+  </xacro:macro>
   <xacro:macro name="pan_tilt_camera_macro" params="namespace parent_link frame_rate
       horizontal_fov image_width image_height image_format min_distance
@@ -176,4 +341,11 @@
     <link name="${namespace}/camera_${camera_suffix}_link">
       <xacro:insert_block name="inertial" />
+      <visual>
+        <origin xyz="0 0 0" rpy="0 0 0" />
+        <geometry>
+          <box size="0.008 0.02 0.012"/>
+        </geometry>
+        <material name="orange"/>
+      </visual>
     </link>
     <joint name="${namespace}/camera_${camera_suffix}_joint" type="fixed">
